File: teensy4_combo_breakout.sch (KiCad schematic (older format))
At the start: 13 parts, among them J1 Conn_01x06, J2 USB_A, U1 TPD3S014

Commit message: First version, ready for fabrication
Parts:
- removed JP?: SolderJumper_2_Open, symbol Jumper:SolderJumper_2_Open
- removed R1: 100k, Resistor_SMD:R_0805_2012Metric_Pad1.15x1.40mm_HandSolder, symbol Device:R_Small_US
- added JP2: Card Detect/29, Jumper:SolderJumper-2_P1.3mm_Bridged_RoundedPad1.0x1.5mm, symbol Jumper:SolderJumper_2_Bridged
- C3: renamed from C?; value C_Small -> 0.1u; footprint (none) -> Capacitor_SMD:C_0805_2012Metric_Pad1.15x1.40mm_HandSolder
- J2: footprint USB_A_Receptacle_SMD_Wuerth_629104190121:USB_A_Receptacle_SMD_Wuerth_629104190121 -> USB_A_Receptacle_SMD_Wuerth_629104190121:USB_A_Receptacle_SMD_Wuerth_629104190121_Narrow
- J3: renamed from J?; footprint (none) -> Connector_PinSocket_2.54mm:PinSocket_1x09_P2.54mm_Vertical
- J4: renamed from J?; footprint (none) -> Connector_Card:microSD_HC_Hirose_DM3D-SF
- JP1: value EN PIN 27 -> Power Enable/27
Connections:
- net D+: now also U1.6 (D2); no longer U1.5 (D1)
- net D-: now also U1.5 (D1); no longer U1.6 (D2)
- net GND: now also C3.1, J3.3 (Pin_3), J4.11 (SHIELD), J4.6 (VSS), J4.9 (DET_B)
- net DAT2: now reaches J3.8 (Pin_8), J4.1 (DAT2)
- net at J4.10 (DET_A): now also JP2.2 (B)
- net DAT3: now reaches J3.7 (Pin_7), J4.2 (DAT3/CD)
- net CMD: now reaches J3.6 (Pin_6), J4.3 (CMD)
- net 3V3: now reaches C3.2, J3.5 (Pin_5), J4.4 (VDD)
- net CLK: now reaches J3.4 (Pin_4), J4.5 (CLK)
- net DAT0: now reaches J3.2 (Pin_2), J4.7 (DAT0)
- net DAT1: now reaches J3.1 (Pin_1), J4.8 (DAT1)
- net 29: now reaches J3.9 (Pin_9)
- net 29: now also JP2.1 (A)
Other:
- moved on the sheet: C1, C2, C3, F1, J1, J2, J3, J4, JP1, L1, U1
